Commit message: 修正URDF模型，修复编译警告

File: src/dog/model/dog.urdf (robot description, URDF)
Before this commit: robot dog, 17 links, 16 joints
Joints:
- joint lb_joint2: origin xyz=-0.00047387 -0.029283 0.059987 rpy=1.5708 -0.67742 -0.016174 -> xyz=-0.00047387 -0.029283 0.059987 rpy=1.5708 0.0 0.0
- joint lb_joint3: origin xyz=0.23001 1.0811E-05 0.0935 rpy=0 0 -1.1563 -> xyz=0.23001 1.0811E-05 0.0935 rpy=0 0 -1.570796325
- joint lb_joint4: origin xyz=0.225 0 0.028 rpy=0 0 2.0497 -> xyz=0.225 0 0.028 rpy=0 0 0
- joint lf_joint2: origin xyz=0 0.029313 0.060013 rpy=-1.5708 0.87219 0 -> xyz=0 0.029313 0.060013 rpy=-1.5708 0.0 0
- joint lf_joint3: origin xyz=0.23001 0 0.0935 rpy=0 0 -1.74 -> xyz=0.23001 0 0.0935 rpy=0 0 -1.570796325
- joint lf_joint4: origin xyz=0.225 0 0.028 rpy=0 0 2.4386 -> xyz=0.225 0 0.028 rpy=0 0 0
- joint rb_joint2: origin xyz=-0.001301 0.029271 0.06 rpy=-1.5708 -0.56823 0.044416 -> xyz=-0.001301 0.029271 0.06 rpy=-1.5708 0 0
- joint rb_joint3: origin xyz=0.23 0 0.0935 rpy=0 0 1.1023 -> xyz=0.23 0 0.0935 rpy=0 0 1.570796325
- joint rb_joint4: origin xyz=0.225 0 0.028 rpy=0 0 1.0368 -> xyz=0.225 0 0.028 rpy=0 0 0
- joint rf_joint2: origin xyz=0 -0.029287 0.059987 rpy=1.5708 0.63231 0 -> xyz=0 -0.029287 0.059987 rpy=1.5708 0.0 0
- joint rf_joint3: origin xyz=0.22999 1.0192E-05 0.0935 rpy=0 0 1.399 -> xyz=0.22999 1.0192E-05 0.0935 rpy=0 0 1.570796325
- joint rf_joint4: origin xyz=0.225 0 0.028 rpy=0 0 0.80414 -> xyz=0.225 0 0.028 rpy=0 0 0

Commit message: 修正模型质量参数

File: src/dog/model/dog.urdf (robot description, URDF)
Before this commit: robot dog, 17 links, 16 joints
Links:
- added link world
- link lb_link4: mass 0.432627590726504 -> 0.65
- link lf_link4: mass 0.392667576355367 -> 0.65
- link rb_link4: mass 0.432627455975141 -> 0.65
- link rf_link4: mass 0.432627569922017 -> 0.65
Joints:
- added joint float_joint: type floating, parent world, child body_link

Commit message: 1

File: src/dog/model/dog.urdf (robot description, URDF)
Before this commit: robot dog, 18 links, 17 joints
Joints:
- joint lb_joint1: limit lower=-3 upper=3 effort=20 velocity=16 -> lower=-4 upper=4 effort=20 velocity=16
- joint lb_joint2: limit lower=-3 upper=3 effort=20 velocity=16 -> lower=-4 upper=4 effort=20 velocity=16
- joint lb_joint3: limit lower=-3 upper=3 effort=20 velocity=16 -> lower=-4 upper=4 effort=20 velocity=16
- joint lf_joint1: limit lower=-3 upper=3 effort=20 velocity=16 -> lower=-4 upper=4 effort=20 velocity=16
- joint lf_joint2: limit lower=-3 upper=3 effort=20 velocity=16 -> lower=-4 upper=4 effort=20 velocity=16
- joint lf_joint3: limit lower=-3 upper=3 effort=20 velocity=16 -> lower=-4 upper=4 effort=20 velocity=16
- joint rb_joint1: limit lower=-3 upper=3 effort=20 velocity=16 -> lower=-4 upper=4 effort=20 velocity=16
- joint rb_joint2: limit lower=-3 upper=3 effort=20 velocity=16 -> lower=-4 upper=4 effort=20 velocity=16
- joint rb_joint3: limit lower=-3 upper=3 effort=20 velocity=16 -> lower=-4 upper=4 effort=20 velocity=16
- joint rf_joint1: limit lower=-3 upper=3 effort=20 velocity=16 -> lower=-4 upper=4 effort=20 velocity=16
- joint rf_joint2: limit lower=-3 upper=3 effort=20 velocity=16 -> lower=-4 upper=4 effort=20 velocity=16
- joint rf_joint3: limit lower=-3 upper=3 effort=20 velocity=16 -> lower=-4 upper=4 effort=20 velocity=16
