Commit message: new_dog_model

File: src/dog2/model/dog2.urdf (robot description, URDF)
Before this commit: robot elephant.SLDASM, 18 links, 17 joints
Links:
- link body_link: geometry collision mesh filename=package://dog2/model/body_link.STL; visual mesh filename=package://dog2/model/body_link.STL
- link lb_link1: mass 0.309387230860269 -> 0.30939; geometry collision mesh filename=package://dog2/model/lb_link1.STL; visual mesh filename=package://dog2/model/lb_link1.STL
- link lb_link2: mass 0.778998090519277 -> 0.779; geometry collision mesh filename=package://dog2/model/lb_link2.STL; visual mesh filename=package://dog2/model/lb_link2.STL
- link lb_link3: mass 0.574756313424315 -> 0.57476; geometry collision mesh filename=package://dog2/model/lb_link3.STL; visual mesh filename=package://dog2/model/lb_link3.STL
- link lb_link4: mass 0.0848322169853741 -> 0.084832; geometry collision mesh filename=package://dog2/model/lb_link4.STL; visual mesh filename=package://dog2/model/lb_link4.STL
- link lf_link1: mass 0.309387230860271 -> 0.30939; geometry collision mesh filename=package://dog2/model/lf_link1.STL; visual mesh filename=package://dog2/model/lf_link1.STL
- link lf_link2: mass 0.778998088622978 -> 0.779; geometry collision mesh filename=package://dog2/model/lf_link2.STL; visual mesh filename=package://dog2/model/lf_link2.STL
- link lf_link3: mass 0.574756313424316 -> 0.57476; geometry collision mesh filename=package://dog2/model/lf_link3.STL; visual mesh filename=package://dog2/model/lf_link3.STL
- link lf_link4: mass 0.0848322169853741 -> 0.084832; geometry collision mesh filename=package://dog2/model/lf_link4.STL; visual mesh filename=package://dog2/model/lf_link4.STL
- link rb_link1: mass 0.309387230860269 -> 0.30939; geometry collision mesh filename=package://dog2/model/rb_link1.STL; visual mesh filename=package://dog2/model/rb_link1.STL
- link rb_link2: mass 0.724056145237142 -> 0.72406; geometry collision mesh filename=package://dog2/model/rb_link2.STL; visual mesh filename=package://dog2/model/rb_link2.STL
- link rb_link3: mass 0.564988657328945 -> 0.56499; geometry collision mesh filename=package://dog2/model/rb_link3.STL; visual mesh filename=package://dog2/model/rb_link3.STL
- link rb_link4: mass 0.084832216985374 -> 0.084832; geometry collision mesh filename=package://dog2/model/rb_link4.STL; visual mesh filename=package://dog2/model/rb_link4.STL
- link rf_link1: mass 0.309387230860329 -> 0.30939; geometry collision mesh filename=package://dog2/model/rf_link1.STL; visual mesh filename=package://dog2/model/rf_link1.STL
- link rf_link2: mass 0.839751446091301 -> 0.72406; geometry collision mesh filename=package://dog2/model/rf_link2.STL; visual mesh filename=package://dog2/model/rf_link2.STL
- link rf_link3: mass 0.574756313424317 -> 0.57476; geometry collision mesh filename=package://dog2/model/rf_link3.STL; visual mesh filename=package://dog2/model/rf_link3.STL
- link rf_link4: mass 0.0848322169853739 -> 0.084832; geometry collision mesh filename=package://dog2/model/rf_link4.STL; visual mesh filename=package://dog2/model/rf_link4.STL
Joints:
- joint lb_joint1: limit lower=-4 upper=4 effort=20 velocity=16 -> lower=0 upper=0 effort=0 velocity=0
- joint lb_joint2: limit lower=-4 upper=4 effort=20 velocity=16 -> lower=0 upper=0 effort=0 velocity=0; origin xyz=0.031313 0 0.06 rpy=1.5708 0.63722 1.5708 -> xyz=0.031313 0 0.06 rpy=1.5708 0 1.5708
- joint lb_joint3: limit lower=-4 upper=4 effort=20 velocity=16 -> lower=0 upper=0 effort=0 velocity=0; origin xyz=0.20707 -0.0041231 0.0726 rpy=0 0 1.2854 -> xyz=0.20707 -0.0041231 0.0726 rpy=0 0 -1.5708
- joint lf_joint1: limit lower=-4 upper=4 effort=20 velocity=16 -> lower=0 upper=0 effort=0 velocity=0
- joint lf_joint2: limit lower=-4 upper=4 effort=20 velocity=16 -> lower=0 upper=0 effort=0 velocity=0; origin xyz=0.031287 0 0.06 rpy=-1.5708 0.46851 -1.5708 -> xyz=0.031287 0 0.06 rpy=-1.5708 0 -1.5708
- joint lf_joint3: limit lower=-4 upper=4 effort=20 velocity=16 -> lower=0 upper=0 effort=0 velocity=0; origin xyz=0.20707 -0.0041231 0.0716 rpy=0 0 -1.7376 -> xyz=0.20707 -0.0041231 0.0716 rpy=0 0 -1.5708
- joint rb_joint1: limit lower=-4 upper=4 effort=20 velocity=16 -> lower=0 upper=0 effort=0 velocity=0
- joint rb_joint2: limit lower=-4 upper=4 effort=20 velocity=16 -> lower=0 upper=0 effort=0 velocity=0; origin xyz=-0.031287 0 0.06 rpy=-1.5708 0.43772 1.5708 -> xyz=-0.031287 0 0.06 rpy=-1.5708 0 1.5708
- joint rb_joint3: limit lower=-4 upper=4 effort=20 velocity=16 -> lower=0 upper=0 effort=0 velocity=0; origin xyz=0.20707 0.0041231 0.0726 rpy=0 0 -0.96369 -> xyz=0.207068955959481 0.00412305443282812 0.0725999999999785 rpy=0 0 1.5708
- joint rf_joint1: limit lower=-4 upper=4 effort=20 velocity=16 -> lower=0 upper=0 effort=0 velocity=0
- joint rf_joint2: limit lower=-4 upper=4 effort=20 velocity=16 -> lower=0 upper=0 effort=0 velocity=0; origin xyz=-0.031313 0 0.06 rpy=1.5708 0.58724 -1.5708 -> xyz=-0.031313 0 0.06 rpy=1.5708 0 -1.5708
- joint rf_joint3: limit lower=-4 upper=4 effort=20 velocity=16 -> lower=0 upper=0 effort=0 velocity=0; origin xyz=0.20707 -0.0041231 0.0726 rpy=0 0 0.92712 -> xyz=0.20707 -0.0041231 0.0726 rpy=0 0 1.5708

Commit message: test2

File: src/dog2/model/dog2.urdf (robot description, URDF)
Before this commit: robot dog2, 18 links, 17 joints
Joints:
- joint lb_joint1: limit lower=0 upper=0 effort=0 velocity=0 -> lower=-4 upper=4 effort=20 velocity=16
- joint lb_joint2: limit lower=0 upper=0 effort=0 velocity=0 -> lower=-4 upper=4 effort=20 velocity=16
- joint lb_joint3: limit lower=0 upper=0 effort=0 velocity=0 -> lower=-4 upper=4 effort=20 velocity=16
- joint lf_joint1: limit lower=0 upper=0 effort=0 velocity=0 -> lower=-4 upper=4 effort=20 velocity=16
- joint lf_joint2: limit lower=0 upper=0 effort=0 velocity=0 -> lower=-4 upper=4 effort=20 velocity=16
- joint lf_joint3: limit lower=0 upper=0 effort=0 velocity=0 -> lower=-4 upper=4 effort=20 velocity=16
- joint rb_joint1: limit lower=0 upper=0 effort=0 velocity=0 -> lower=-4 upper=4 effort=20 velocity=16
- joint rb_joint2: limit lower=0 upper=0 effort=0 velocity=0 -> lower=-4 upper=4 effort=20 velocity=16
- joint rb_joint3: limit lower=0 upper=0 effort=0 velocity=0 -> lower=-4 upper=4 effort=20 velocity=16
- joint rf_joint1: limit lower=0 upper=0 effort=0 velocity=0 -> lower=-4 upper=4 effort=20 velocity=16
- joint rf_joint2: limit lower=0 upper=0 effort=0 velocity=0 -> lower=-4 upper=4 effort=20 velocity=16
- joint rf_joint3: limit lower=0 upper=0 effort=0 velocity=0 -> lower=-4 upper=4 effort=20 velocity=16

Commit message: 新狗的urdf模型

File: src/dog2/model/dog2.urdf (robot description, URDF)
Before this commit: robot dog2, 18 links, 17 joints
Links:
- link body_link: mass 2.2266 -> 4.829; geometry collision mesh filename=package://dog2/model/body_link.stl; visual mesh filename=package://dog2/model/body_link.stl
- link lb_link1: mass 0.30939 -> 0.676831591069983; geometry collision mesh filename=package://dog2/model/lb_link1.stl; visual mesh filename=package://dog2/model/lb_link1.stl
- link lb_link2: mass 0.779 -> 1.40828094682296; geometry collision mesh filename=package://dog2/model/lb_link2.stl; visual mesh filename=package://dog2/model/lb_link2.stl
- link lb_link3: mass 0.57476 -> 0.466427846899075; geometry collision mesh filename=package://dog2/model/lb_link3.stl; visual mesh filename=package://dog2/model/lb_link3.stl
- link lb_link4: mass 0.084832 -> 0.084832216985374; geometry collision mesh filename=package://dog2/model/lb_link4.stl; visual mesh filename=package://dog2/model/lb_link4.stl
- link lf_link1: mass 0.30939 -> 0.676831582353488; geometry collision mesh filename=package://dog2/model/lf_link1.stl; visual mesh filename=package://dog2/model/lf_link1.stl
- link lf_link2: mass 0.779 -> 1.40828092509435; geometry collision mesh filename=package://dog2/model/lf_link2.stl; visual mesh filename=package://dog2/model/lf_link2.stl
- link lf_link3: mass 0.57476 -> 0.466427846899075; geometry collision mesh filename=package://dog2/model/lf_link3.stl; visual mesh filename=package://dog2/model/lf_link3.stl
- link lf_link4: mass 0.084832 -> 0.084832216985374; geometry collision mesh filename=package://dog2/model/lf_link4.stl; visual mesh filename=package://dog2/model/lf_link4.stl
- link rb_link1: mass 0.30939 -> 0.676831591069986; geometry collision mesh filename=package://dog2/model/rb_link1.stl; visual mesh filename=package://dog2/model/rb_link1.stl
- link rb_link2: mass 0.72406 -> 1.35333899025955; geometry collision mesh filename=package://dog2/model/rb_link2.stl; visual mesh filename=package://dog2/model/rb_link2.stl
- link rb_link3: mass 0.56499 -> 0.456660190803704; geometry collision mesh filename=package://dog2/model/rb_link3.stl; visual mesh filename=package://dog2/model/rb_link3.stl
- link rb_link4: mass 0.084832 -> 0.084832216985374; geometry collision mesh filename=package://dog2/model/rb_link4.stl; visual mesh filename=package://dog2/model/rb_link4.stl
- link rf_link1: mass 0.30939 -> 0.677615723872956; geometry collision mesh filename=package://dog2/model/rf_link1.stl; visual mesh filename=package://dog2/model/rf_link1.stl
- link rf_link2: mass 0.72406 -> 1.35333898941377; geometry collision mesh filename=package://dog2/model/rf_link2.stl; visual mesh filename=package://dog2/model/rf_link2.stl
- link rf_link3: mass 0.57476 -> 0.466427846899075; geometry collision mesh filename=package://dog2/model/rf_link3.stl; visual mesh filename=package://dog2/model/rf_link3.stl
- link rf_link4: mass 0.084832 -> 0.0848322169853742; geometry collision mesh filename=package://dog2/model/rf_link4.stl; visual mesh filename=package://dog2/model/rf_link4.stl
Joints:
- joint lb_joint1: limit lower=-4 upper=4 effort=20 velocity=16 -> lower=-3.14159 upper=3.14159 effort=23 velocity=30; origin xyz=-0.1966 0.059987 0.042001 rpy=-1.5708 0 1.5708 -> xyz=-0.20677 0.058639 0.03776 rpy=-1.5708 0 1.5708
- joint lb_joint2: limit lower=-4 upper=4 effort=20 velocity=16 -> lower=-3.14159 upper=3.14159 effort=23 velocity=30; origin xyz=0.031313 0 0.06 rpy=1.5708 0 1.5708 -> xyz=0.029301 -1.3226E-05 0.06 rpy=1.5708 0 1.5708
- joint lb_joint3: limit lower=-4 upper=4 effort=20 velocity=16 -> lower=-3.14159 upper=3.14159 effort=23 velocity=30; origin xyz=0.20707 -0.0041231 0.0726 rpy=0 0 -1.5708 -> xyz=0.20711 0 0.0746 rpy=0 0 -1.570796
- joint lb_joint4: axis 0 0 1 -> 0 0 0
- joint lf_joint1: limit lower=-4 upper=4 effort=20 velocity=16 -> lower=-3.14159 upper=3.14159 effort=23 velocity=30; origin xyz=0.1966 0.060013 0.042001 rpy=1.5708 0 1.5708 -> xyz=0.18433 0.058364 0.045534 rpy=1.5708 0 1.5708
- joint lf_joint2: limit lower=-4 upper=4 effort=20 velocity=16 -> lower=-3.14159 upper=3.14159 effort=23 velocity=30; origin xyz=0.031287 0 0.06 rpy=-1.5708 0 -1.5708 -> xyz=0.031298 0.00022929 0.06 rpy=-1.5708 0 -1.5708
- joint lf_joint3: limit lower=-4 upper=4 effort=20 velocity=16 -> lower=-3.14159 upper=3.14159 effort=23 velocity=30; origin xyz=0.20707 -0.0041231 0.0716 rpy=0 0 -1.5708 -> xyz=0.20707 -0.0041231 0.0716 rpy=0 0 -1.570796
- joint rb_joint1: limit lower=-4 upper=4 effort=20 velocity=16 -> lower=-3.14159 upper=3.14159 effort=23 velocity=30; origin xyz=-0.1966 -0.060013 0.042001 rpy=-1.5708 0 1.5708 -> xyz=-0.20677 -0.06136 0.037786 rpy=-1.5708 0 1.5708
- joint rb_joint2: limit lower=-4 upper=4 effort=20 velocity=16 -> lower=-3.14159 upper=3.14159 effort=23 velocity=30; origin xyz=-0.031287 0 0.06 rpy=-1.5708 0 1.5708 -> xyz=-0.029301 1.3226E-05 0.06 rpy=-1.5708 0 1.5708
- joint rb_joint3: limit lower=-4 upper=4 effort=20 velocity=16 -> lower=-3.14159 upper=3.14159 effort=23 velocity=30; origin xyz=0.207068955959481 0.00412305443282812 0.0725999999999785 rpy=0 0 1.5708 -> xyz=0.20711 0 0.0746 rpy=0 0 1.570796
- joint rb_joint4: origin xyz=0.22 0 0 rpy=-3.1416 0 -1.5708 -> xyz=0.22 0 0 rpy=3.1416 0 -1.5708
- joint rf_joint1: limit lower=-4 upper=4 effort=20 velocity=16 -> lower=-3.14159 upper=3.14159 effort=23 velocity=30; origin xyz=0.1966 -0.059987 0.042001 rpy=1.5708 0 1.5708 -> xyz=0.18643 -0.06136 0.03776 rpy=1.5708 0 1.5708
- joint rf_joint2: limit lower=-4 upper=4 effort=20 velocity=16 -> lower=-3.14159 upper=3.14159 effort=23 velocity=30; origin xyz=-0.031313 0 0.06 rpy=1.5708 0 -1.5708 -> xyz=-0.0313 -0.00018614 0.06 rpy=1.5708 0 -1.5708
- joint rf_joint3: limit lower=-4 upper=4 effort=20 velocity=16 -> lower=-3.14159 upper=3.14159 effort=23 velocity=30
